File: pcb/glowcost-geiger.kicad_pcb (KiCad board)
At the start: 2 copper layers, 120 x 32 mm, 79 parts, among them J1 JST GH 4-pin, J2 C142864 DNP, J3 C142864 DNP, Q1 MMBT3904LT1G, Q2 MMBT3904LT1G, U1 TLC555IDR, U2 MCP6562T-E/MS

Commit message: Update the board for the SBM-20 and the firmware faults.
J2 and J3 are both C19184098. The ATtiny, boost switch, and STEMMA QT connectors sit on a bay added along the lower edge. Multiplier copper that still matched the sheet was kept; the new nets are not fully routed. Fault traces follow the PA6 trip and the 20% latch.
Parts:
- removed C10: 10 pF, glowcost:C_OV
- removed J1: JST GH 4-pin, glowcost:J1
- removed R10: 33 MR, glowcost:R_OV1
- removed R12: 33 MR, glowcost:R_OV2
- removed R14: 33 MR, glowcost:R_OV3
- removed R16: 33 MR, glowcost:R_OV4
- removed R18: 402 kR, glowcost:R_OVBOT
- removed R9: 100 kR, glowcost:R_EN
- removed TP11: P1, glowcost:TP11
- removed TP12: S1, glowcost:TP12
- removed TP13: P2, glowcost:TP13
- removed TP14: S2, glowcost:TP14
- removed TP15: P3, glowcost:TP15
- removed TP16: S3, glowcost:TP16
- removed TP17: P4, glowcost:TP17
- removed TP18: S4, glowcost:TP18
- removed TP20: OVP, glowcost:TP20
- removed TP22: GND, glowcost:TP22
- removed TP3: EN, glowcost:TP3
- removed TP5: DRIVE, glowcost:TP5
- removed TP7: COLLECTOR, glowcost:TP7
- removed TP9: GND, glowcost:TP9
- removed U2: MCP6562T-E/MS, U2
- added C11: 100 nF, C_0603_1608Metric, F.Cu at (118.0, 122.0)
- added J4: SM04B-SRSS-TB / C160404, JST_SH_SM04B-SRSS-TB_1x04-1MP_P1.00mm_Horizontal, F.Cu at (52.0, 124.0)
- added J5: SM04B-SRSS-TB / C160404, JST_SH_SM04B-SRSS-TB_1x04-1MP_P1.00mm_Horizontal, F.Cu at (70.0, 124.0)
- added JP2: A0 open=high, SJ_LED, F.Cu at (86.0, 124.0)
- added JP3: A1 open=high, SJ_LED, F.Cu at (94.0, 124.0)
- added L1: 1 mH YNR6045-102M, L_6.3x6.3_H3, F.Cu at (154.0, 123.0)
- added Q3: TN2404K / C468011, SOT-23, F.Cu at (144.0, 123.0)
- added R25: 220 R, R_OUT, F.Cu at (136.0, 126.0)
- added R26: 4.7 kR, R_OUT, F.Cu at (124.0, 126.0)
- added R27: 4.7 kR, R_OUT, F.Cu at (130.0, 126.0)
- added TP24: UPDI, TP1, F.Cu at (112.0, 128.0)
- added TP28: UART_TX, TP1, F.Cu at (104.0, 128.0)
- J2: value C142864 DNP -> C19184098; footprint glowcost:J2 -> MY-AA-03
- J3: value C142864 DNP -> C19184098; footprint glowcost:J3 -> MY-AA-03
- U1: value TLC555IDR -> ATTINY1616-MNR / C507118; footprint U1 -> VQFN-20-1EP_3x3mm_P0.4mm_EP1.7x1.7mm
- moved U1 188.8 mm to (108.0, 122.0)
- moved R13 69.8 mm to (78.0, 128.0)
- moved R15 57.3 mm to (88.0, 128.0)
- moved R23 44.0 mm to (96.0, 128.0)
- moved R21 12.2 mm to (58.0, 112.0)
- moved H1 12.0 mm to (44.0, 128.0)
- moved H3 12.0 mm to (156.0, 128.0)
- moved J2 5.50 mm to (158.0, 100.0), turned to -90 degrees
- moved J3 5.50 mm to (42.0, 100.0), turned to 90 degrees
- turned D1 to -90 degrees
- turned D10 to 180 degrees
- turned D2 to -90 degrees
- turned D3 to -90 degrees
- turned D4 to -90 degrees
- turned D5 to -90 degrees
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Connections:
- net /ANODE_MID renamed Net-(R19-Pad2)
- net /BL1 renamed Net-(R11-Pad2)
- net /BL2 renamed Net-(R13-Pad2)
- net /BL3 renamed Net-(R15-Pad2)
- net /DIV1 renamed Net-(R1-Pad2)
- net /DIV2 renamed Net-(R2-Pad2)
- net /DIV3 renamed Net-(R3-Pad2)
- net /LED_BASE renamed Net-(Q2-B)
- C8 pad 2: /S4 -> /HV
- D1 pad 1: GND -> /P1
- D1 pad 2: /P1 -> GND
- D10 pad 1: GND -> /BASE
- D10 pad 2: /BASE -> GND
- D2 pad 1: /P1 -> /S1
- D2 pad 2: /S1 -> /P1
- D3 pad 1: /S1 -> /P2
- D3 pad 2: /P2 -> /S1
- D4 pad 1: /P2 -> /S2
- D4 pad 2: /S2 -> /P2
- D5 pad 1: /S2 -> /P3
- D5 pad 2: /P3 -> /S2
- D6 pad 1: /P3 -> /S3
- D6 pad 2: /S3 -> /P3
- D7 pad 1: /S3 -> /P4
- D7 pad 2: /P4 -> /S3
- D8 pad 1: /P4 -> /HV
- D8 pad 2: /S4 -> /P4
- D9 pad 1: /LED_A -> Net-(D9-K)
- D9 pad 2: /LED_K -> Net-(D9-A)
- JP1 pad 2: /LED_SUPPLY -> Net-(JP1-B)
- Q2 pad 3: /LED_K -> Net-(D9-K)
- R1 pad 1: /S4 -> /HV
- R11 pad 1: /S4 -> /HV
- R19 pad 1: /S4 -> /HV
- R24 pad 1: /DRIVE -> /COLLECTOR
- R6 pad 1: /LED_SUPPLY -> Net-(D9-A)
- R6 pad 2: /LED_A -> Net-(JP1-B)
- R7 pad 1: /DRIVE -> /COLLECTOR
- U1 pad 1: (no net) -> /COLLECTOR
- U1 pad 2: (no net) -> unconnected-(U1-PA3-Pad2)
- U1 pad 3: (no net) -> GND
- U1 pad 4: (no net) -> V3V3
- U1 pad 5: (no net) -> unconnected-(U1-PA4-Pad5)
- U1 pad 6: (no net) -> unconnected-(U1-PA5-Pad6)
- U1 pad 7: (no net) -> /SENSE
- U1 pad 8: (no net) -> unconnected-(U1-PA7-Pad8)
Routing:
- net /S4: track 53.8 -> 0.00 mm, vias 2 -> 0
- net /DRIVE: track 50.3 -> 0.00 mm, vias 1 -> 0
- net /COLLECTOR: track 17.2 -> 67.5 mm, vias 1 -> 2
- net V3V3: track 44.3 -> 0.00 mm, vias 2 -> 0
- net /P4: track 31.8 -> 0.00 mm
- net /LED_K: track 25.4 -> 0.00 mm
- net /OV2: track 20.4 -> 0.00 mm
- net /OV1: track 19.6 -> 0.00 mm
- net Net-(R3-Pad2): track 18.9 -> 0.00 mm, vias 2 -> 0
- net /OV3: track 18.7 -> 0.00 mm, vias 2 -> 0
- net Net-(R1-Pad2): track 18.7 -> 0.00 mm, vias 2 -> 0
- net GND: track 184.0 -> 168.0 mm
- net /OVP: track 15.7 -> 0.00 mm, vias 1 -> 0
- net /TTL: track 24.3 -> 13.2 mm
- net /EN: track 9.87 -> 0.00 mm, vias 1 -> 0
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Other:
- board size 120 x 32 mm -> 120 x 48 mm
- board text removed: "3V3 GND PULSE EN"
- board text removed: "ANALOG - NO MCU"
- board text removed: "HEIGHT TBD"
- board text removed: "TP11 P1"
- board text removed: "TP12 S1"
- board text removed: "TP13 P2"
- board text removed: "TP14 S2"
- board text removed: "TP15 P3"
- board text removed: "TP16 S3"
- board text removed: "TP17 P4"
- board text removed: "TP18 S4"
- board text removed: "TP20 OVP"
- board text removed: "TP22 GND"
- board text removed: "TP3 EN"
- board text removed: "TP5 DRIVE"
- board text removed: "TP7 COLLECTOR"
- board text removed: "TP9 GND"
- board text removed: "U1/U2 RESERVE"
