File: pcb/glowcost-geiger.kicad_sch (KiCad schematic)
At the start: 83 parts, among them J1 JST GH 4-pin, J2 C142864 DNP, J3 C142864 DNP, J4 SM04B-SRSS-TB / C160404, J5 SM04B-SRSS-TB / C160404, Q1 MMBT3904LT1G, Q2 MMBT3904LT1G, Q3 HL2310A / C7420347, U1 ATTINY1616-MNR / C507118

Commit message: Organize schematic like x.drop-beacon
Beacon-style A2 frames and section titles, DESIGN NOTES column, and a filled
title block. Connectivity unchanged; ERC still 0 errors.
Other:
- note added: "ARCHITECTURE ATtiny1616-only: MCU PWM drives HV boost, counts pulses, serves I2C, reads A0/A1 and HV/3V3 ADC. No TLC555 / MCP6562. Raw TTL pulse path stays hardware."
- note added: "BOOST / HV Q3 HL2310A (1=G 2=S 3=D); R25 gate. L1 1 mH — watch DCR (~9.5 R). C1–C8: 10nF C0G 630V 1206. D1–D8: BAV21W. SW ~106 Vpk; S4 ~399 V."
- note added: "DESIGN NOTES"
- note added: "OUTPUT / LED"
- note added: "OVP / PULSE / TUBE"
- note added: "PIN MAP — U1 PA2 COLLECTOR PA4 SDA PA5 SCL PA6 SENSE (HV) PA7 V3V3_SENSE PB0 A0 PB1 A1 PB2 HV_PWM PB3 EN PA0 UPDI PA1 UART_TX (USART0 alt) Default USART0 TX is PB2 — remapped."
- note added: "PROBE ACCESS"
- note added: "SAFETY / FAB 400 V on tube clips / HV nodes. Discharge before handling. PCB: known DRC issues — prototype only. Clips C142864 DNP; fit after assembly. Run ERC; human-review HV creepage."
- note added: "STEMMA QT / ADDRESS J4/J5 JST-SH: 1=GND 2=3V3 3=SDA 4=SCL JP2/JP3 open = 0x2F; bridge = low bit. One pull-up set per bus segment."
- note removed: "399.16 V = 1.242 x (132M + 412k) / 412k 3.02 uA at 400 V; C9 time constant ~41 us."
- note removed: "400 V present on exposed pads / tube clips. Discharge and verify before handling. Do not connect ordinary Pi / scope probes to HV. Preserved routing has unresolved clearances. U1/U2 have no physical implementation. This is NOT a fabrication release. 22 plated probe holes; 1 mm drill / 2 mm pads. See README for model limits and DRC report."
- note removed: "ATtiny-only: MCU PWM boost + pulse/I2C/ADC. No 555/MCP6562. Dual STEMMA J4/J5."
- note removed: "C1-C8: 10nF C0G 630V 1206. D1-D8: BAV21W-7-F. SW~106Vpk; S4~399V nom."
- note removed: "CTRL"
- note removed: "DRIVE merged into COLLECTOR. No TLC555/MCP6562."
- note removed: "Factory copper bridge: cut to disable; solder to restore. ~1.28 mA LED during pulse. Q_LED buffers DRIVE. No pulse stretching; flashes may be hard to see."
- note removed: "HV"
- note removed: "HV / TUBE / PULSE"
- note removed: "HV LADDER"
- note removed: "Independent OVP divider; verify diode reverse stress/leakage."
- note removed: "JP2/JP3: leave OPEN for 0x2F; bridge to GND for low"
- note removed: "NOTES"
- note removed: "OVP"
- note removed: "OVP / PULSE"
- note removed: "PA2=COLLECTOR PA4=SDA PA5=SCL PA6=SENSE PA7=V3V3_SENSE"
- note removed: "PB0=A0 PB1=A1 PB2=HV_PWM PB3=EN PA0=UPDI PA1=UART_TX (USART0 alt)"
- note removed: "PI"
- note removed: "PI J1: 1=3V3 2=GND 3=PULSE 4=EN"
- note removed: "PIN MAP (U1)"
- note removed: "PROBE STRIP"
- note removed: "PROBES"
- note removed: "PROG"
- note removed: "PWR"
- note removed: "Q3 HL2310A (1=G 2=S 3=D); R25 gate; L1 1mH DCR 9.5R (efficiency risk)."
- note removed: "R_A1/R_A2: 2.49 MR EACH, >=500 V working rating; ~88.4 uA maximum at 440 V. J2/J3: C142864 DNP for JLC, hand-fit clips. Tube supplied by user. U2 inverts Q1 and blanks on EN / HV-ready / OVP. No MCU. Physical logic remains unfinished. Plan 250 us tube dead time (reference ~190 us); dose conversion is approximate."
- note removed: "STEMMA QT JST SH 1=GND 2=V+ 3=SDA 4=SCL"
- note removed: "UPDI / UART pads"
- title: Glowcost Geiger - prototype conversion -> gLowCost-geiger
Changed lines of the file:
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@@
+(kicad_sch (version 20250114) (generator "eeschema") (paper A2) (title_block
+		(title "gLowCost-geiger")
+		(date "2026-09-19")
+		(rev "ATtiny1616")
+		(company "muonTelescope")
+		(comment 1 "Sawaiz Syed")
+		(comment 2 "Prototype — HV not fab-qualified")
+	(rectangle (start 18 18) (end 90 80)
+		(stroke (width 0.2) (type default))
+		(fill (type none))
+	)
+	(text "PI HEADER" (at 20 20 0)
+		(effects (font (size 1.3 1.3)) (justify left top))
+	)
+	(rectangle (start 92 18) (end 145 95)
+		(stroke (width 0.2) (type default))
+		(fill (type none))
+	)
+	(text "MCU" (at 94 20 0)
+		(effects (font (size 1.3 1.3)) (justify left top))
+	)
+	(rectangle (start 145 12) (end 210 75)
+		(stroke (width 0.2) (type default))
+		(fill (type none))
+	)
+	(text "BOOST" (at 147 14 0)
+		(effects (font (size 1.3 1.3)) (justify left top))
+	)
+	(rectangle (start 18 88) (end 115 165)
+		(stroke (width 0.2) (type default))
+		(fill (type none))
+	)
+	(text "STEMMA / I2C" (at 20 90 0)
+		(effects (font (size 1.3 1.3)) (justify left top))
+	)
+	(rectangle (start 125 78) (end 300 165)
+		(stroke (width 0.2) (type default))
+		(fill (type none))
+	)
+	(text "HV MULTIPLIER" (at 127 80 0)
+		(effects (font (size 1.3 1.3)) (justify left top))
+	)
+	(rectangle (start 18 170) (end 300 255)
+		(stroke (width 0.2) (type default))
+		(fill (type none))
+	)
+	(text "OVP / PULSE / TUBE" (at 20 172 0)
+		(effects (font (size 1.3 1.3)) (justify left top))
+	)
+	(rectangle (start 305 18) (end 420 165)
+		(stroke (width 0.2) (type default))
+		(fill (type none))
+	)
+	(text "OUTPUT / LED" (at 307 20 0)
+		(effects (font (size 1.3 1.3)) (justify left top))
+	)
+	(rectangle (start 18 258) (end 220 295)
+		(stroke (width 0.2) (type default))
+		(fill (type none))
+	)
+	(text "PROBE ACCESS" (at 20 260 0)
+		(effects (font (size 1.3 1.3)) (justify left top))
+	)
+	(rectangle (start 425 15) (end 560 300)
+		(stroke (width 0.2) (type default))
+		(fill (type none))
+	)
+	(text "DESIGN NOTES" (at 427 17 0)
+		(effects (font (size 1.3 1.3)) (justify left top))
+	)
+	(text "ARCHITECTURE\n\nATtiny1616-only: MCU PWM drives HV boost,\ncounts pulses, serves I2C, reads A0/A1 and\nHV/3V3 ADC. No TLC555 / MCP6562.\nRaw TTL pulse path stays hardware." (at 430 22 0)
+		(effects (font (size 1.27 1.27)) (justify left top))
+	)
+	(text "PIN MAP — U1\n\nPA2 COLLECTOR   PA4 SDA   PA5 SCL\nPA6 SENSE (HV)  PA7 V3V3_SENSE\nPB0 A0   PB1 A1   PB2 HV_PWM   PB3 EN\nPA0 UPDI   PA1 UART_TX (USART0 alt)\nDefault USART0 TX is PB2 — remapped." (at 430 72 0)
+		(effects (font (size 1.27 1.27)) (justify left top))
+	)
+	(text "STEMMA QT / ADDRESS\n\nJ4/J5 JST-SH: 1=GND 2=3V3 3=SDA 4=SCL\nJP2/JP3 open = 0x2F; bridge = low bit.\nOne pull-up set per bus segment." (at 430 132 0)
+		(effects (font (size 1.27 1.27)) (justify left top))
+	)
+	(text "BOOST / HV\n\nQ3 HL2310A (1=G 2=S 3=D); R25 gate.\nL1 1 mH — watch DCR (~9.5 R).\nC1–C8: 10nF C0G 630V 1206.\nD1–D8: BAV21W. SW ~106 Vpk; S4 ~399 V." (at 430 178 0)
+		(effects (font (size 1.27 1.27)) (justify left top))
+	)
+	(text "SAFETY / FAB\n\n400 V on tube clips / HV nodes.\nDischarge before handling.\nPCB: known DRC issues — prototype only.\nClips C142864 DNP; fit after assembly.\nRun ERC; human-review HV creepage." (at 430 238 0)
+		(effects (font (size 1.27 1.27)) (justify left top))
+	)
+)

Commit message: Fix tube anode/cathode nets, refresh SPICE, document electrical review
Reattach R20 to ANODE and R21/R22 to CATHODE after layout cleanup left
them floating. Point simulate.py at docs/sim, annotate the ATtiny-PWM
deck, and update the README with review notes plus sim diagrams.
Connections:
- net ANODE: now also GM1.1, R20.2
- net CATHODE: now also GM1.2, R21.1, R22.1
Changed lines of the file:
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@@
-(kicad_sch (version 20250114) (generator "eeschema") (paper A2) (title_block
-		(title "gLowCost-geiger")
-		(date "2026-09-19")
-		(rev "ATtiny1616")
-		(company "muonTelescope")
-		(comment 1 "Sawaiz Syed")
-		(comment 2 "Prototype — HV not fab-qualified")
-	(rectangle (start 18 18) (end 90 80)
-		(stroke (width 0.2) (type default))
-		(fill (type none))
-	)
-	(text "PI HEADER" (at 20 20 0)
-		(effects (font (size 1.3 1.3)) (justify left top))
-	)
-	(rectangle (start 92 18) (end 145 95)
-		(stroke (width 0.2) (type default))
-		(fill (type none))
-	)
-	(text "MCU" (at 94 20 0)
-		(effects (font (size 1.3 1.3)) (justify left top))
-	)
-	(rectangle (start 145 12) (end 210 75)
-		(stroke (width 0.2) (type default))
-		(fill (type none))
-	)
-	(text "BOOST" (at 147 14 0)
-		(effects (font (size 1.3 1.3)) (justify left top))
-	)
-	(rectangle (start 18 88) (end 115 165)
-		(stroke (width 0.2) (type default))
-		(fill (type none))
-	)
-	(text "STEMMA / I2C" (at 20 90 0)
-		(effects (font (size 1.3 1.3)) (justify left top))
-	)
-	(rectangle (start 125 78) (end 300 165)
-		(stroke (width 0.2) (type default))
-		(fill (type none))
-	)
-	(text "HV MULTIPLIER" (at 127 80 0)
-		(effects (font (size 1.3 1.3)) (justify left top))
-	)
-	(rectangle (start 18 170) (end 300 255)
-		(stroke (width 0.2) (type default))
-		(fill (type none))
-	)
-	(text "OVP / PULSE / TUBE" (at 20 172 0)
-		(effects (font (size 1.3 1.3)) (justify left top))
-	)
-	(rectangle (start 305 18) (end 420 165)
-		(stroke (width 0.2) (type default))
-		(fill (type none))
-	)
-	(text "OUTPUT / LED" (at 307 20 0)
-		(effects (font (size 1.3 1.3)) (justify left top))
-	)
-	(rectangle (start 18 258) (end 220 295)
-		(stroke (width 0.2) (type default))
-		(fill (type none))
-	)
-	(text "PROBE ACCESS" (at 20 260 0)
-		(effects (font (size 1.3 1.3)) (justify left top))
-	)
-	(rectangle (start 425 15) (end 560 300)
-		(stroke (width 0.2) (type default))
-		(fill (type none))
-	)
-	(text "DESIGN NOTES" (at 427 17 0)
-		(effects (font (size 1.3 1.3)) (justify left top))
-	)
-	(text "ARCHITECTURE\n\nATtiny1616-only: MCU PWM drives HV boost,\ncounts pulses, serves I2C, reads A0/A1 and\nHV/3V3 ADC. No TLC555 / MCP6562.\nRaw TTL pulse path stays hardware." (at 430 22 0)
-		(effects (font (size 1.27 1.27)) (justify left top))
-	)
-	(text "PIN MAP — U1\n\nPA2 COLLECTOR   PA4 SDA   PA5 SCL\nPA6 SENSE (HV)  PA7 V3V3_SENSE\nPB0 A0   PB1 A1   PB2 HV_PWM   PB3 EN\nPA0 UPDI   PA1 UART_TX (USART0 alt)\nDefault USART0 TX is PB2 — remapped." (at 430 72 0)
-		(effects (font (size 1.27 1.27)) (justify left top))
-	)
-	(text "STEMMA QT / ADDRESS\n\nJ4/J5 JST-SH: 1=GND 2=3V3 3=SDA 4=SCL\nJP2/JP3 open = 0x2F; bridge = low bit.\nOne pull-up set per bus segment." (at 430 132 0)
-		(effects (font (size 1.27 1.27)) (justify left top))
-	)
-	(text "BOOST / HV\n\nQ3 HL2310A (1=G 2=S 3=D); R25 gate.\nL1 1 mH — watch DCR (~9.5 R).\nC1–C8: 10nF C0G 630V 1206.\nD1–D8: BAV21W. SW ~106 Vpk; S4 ~399 V." (at 430 178 0)
-		(effects (font (size 1.27 1.27)) (justify left top))
-	)
-	(text "SAFETY / FAB\n\n400 V on tube clips / HV nodes.\nDischarge before handling.\nPCB: known DRC issues — prototype only.\nClips C142864 DNP; fit after assembly.\nRun ERC; human-review HV creepage." (at 430 238 0)
-		(effects (font (size 1.27 1.27)) (justify left top))
-	)
-)

Commit message: Swap L1 to YNR6045-102M and add firmware SENSE OVP
Replace B82442T1105K050 (9.5 Ω DCR, wrong 1210 footprint) with
YNR6045-102M / C497845 (4.5 Ω, 6×6 mm, 300 mA Isat). SPICE DCR=4.5;
suite re-passed. Firmware drives HV_PWM with soft-start and clamps via
PA6 SENSE (~420 V trip / ~390 V recover) since no hardware OVP remains.
Parts:
- L1: value 1 mH B82442T1105K050 -> 1 mH YNR6045-102M; footprint Inductor_SMD:L_1210_3225Metric -> Inductor_SMD:L_6.3x6.3_H3; LCSC C2041861 -> C497845; MPN B82442T1105K050 -> YNR6045-102M

Commit message: Document MCU HV duty range and sense readback.
PWM at 1 µA spans about 37 V at 1% duty to 604 V at 20%, 1.5 V per timer count, and the 60 V FET limit lands near 233 V. PA6 readback is 1.04 V per count. The L1 sheet note now matches YNR6045-102M.
Connections:
- net BASE: no longer Q1.1 (B), R22.2
- new net: Q1.1 (B), R22.2
Other:
- note added: "BOOST / HV Q3 HL2310A (1=G 2=S 3=D); R25 gate. L1 YNR6045-102M 1 mH, DCR 4.5 R. C1–C8: 10nF C0G 630V 1206. D1–D8: BAV21W. SW ~106 Vpk; S4 ~399 V."
- note removed: "BOOST / HV Q3 HL2310A (1=G 2=S 3=D); R25 gate. L1 1 mH — watch DCR (~9.5 R). C1–C8: 10nF C0G 630V 1206. D1–D8: BAV21W. SW ~106 Vpk; S4 ~399 V."
- moved on the sheet: D9, GM1, J2, J3, JP1, Q1, R11, R13, R15, R17, R19, R20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

Commit message: Redraw the ATtiny sheet and publish the rerun HV charts.
Move TWI to PB1/PB0, drop the Pi header and the unused dividers, and rate Q3 as the 240 V TN2404K. The ngspice suite was rerun; the README is the current schematic crops and the new duty, startup, and readback charts.
Parts:
- removed C10: 10 pF, glowcost:C_OV, symbol Glowcost:C
- removed J1: JST GH 4-pin, glowcost:J1, symbol Glowcost:Conn_01x04
- removed R10: 33 MR, glowcost:R_OV1, symbol Glowcost:R_Small_US
- removed R12: 33 MR, glowcost:R_OV2, symbol Glowcost:R_Small_US
- removed R14: 33 MR, glowcost:R_OV3, symbol Glowcost:R_Small_US
- removed R16: 33 MR, glowcost:R_OV4, symbol Glowcost:R_Small_US
- removed R18: 402 kR, glowcost:R_OVBOT, symbol Glowcost:R_Small_US
- removed R28, R29: 10 kR, glowcost:R1, symbol Glowcost:R_Small_US
- removed R9: 100 kR, glowcost:R_EN, symbol Glowcost:R_Small_US
- removed TP20: OVP, glowcost:TP20, symbol Glowcost:TestPoint
- removed TP22: GND, glowcost:TP22, symbol Glowcost:TestPoint
- removed TP23: V3V3, glowcost:TP1, symbol Glowcost:TestPoint
- removed TP25, TP29: GND, glowcost:TP1, symbol Glowcost:TestPoint
- removed TP3: EN, glowcost:TP3, symbol Glowcost:TestPoint
- removed TP5: DRIVE, glowcost:TP5, symbol Glowcost:TestPoint
- removed TP7: COLLECTOR, glowcost:TP7, symbol Glowcost:TestPoint
- removed TP9: GND, glowcost:TP9, symbol Glowcost:TestPoint
- Q3: value HL2310A / C7420347 -> TN2404K / C468011; symbol Glowcost:HL2310A -> Glowcost:TN2404K; LCSC C7420347 -> C468011; MPN HL2310A -> TN2404K-T1-GE3
- R25: footprint glowcost:R1 -> glowcost:R_OUT
- R26, R27: footprint glowcost:R1 -> glowcost:R_OUT; MPN FRG2512F3305TS -> 0603WAF4701T5E
Connections:
- net A0: now also U1.15 (PC0); no longer U1.14 (PB0)
- net A1: now also U1.16 (PC1); no longer U1.13 (PB1)
- net BASE: now also D10.1 (K), Q1.1 (B), R22.2; no longer D10.2 (K)
- net GND: now also D1.2 (A), D10.2 (A); no longer D1.1 (A), D10.1 (A)
- net P1: now also D1.1 (K), D2.2 (A); no longer D1.2 (K), D2.1 (A)
- net P2: now also D3.1 (K), D4.2 (A); no longer D3.2 (K), D4.1 (A)
- net P3: now also D5.1 (K), D6.2 (A); no longer D5.2 (K), D6.1 (A)
- net P4: now also D7.1 (K), D8.2 (A); no longer D7.2 (K), D8.1 (A)
- net S1: now also D2.1 (K), D3.2 (A); no longer D2.2 (K), D3.1 (A)
- net S2: now also D4.1 (K), D5.2 (A); no longer D4.2 (K), D5.1 (A)
- net S3: now also D6.1 (K), D7.2 (A); no longer D6.2 (K), D7.1 (A)
- net SCL: now also U1.14 (PB0); no longer U1.6 (PA5)
- net SDA: now also U1.13 (PB1); no longer U1.5 (PA4)
- net at D9.1 (K): now also Q2.3 (C); no longer R6.2
- net at R6.1: now also D9.2 (A); no longer JP1.2 (B)
- net EN: no longer names the net of U1.11 (PB3)
- net GATE: no longer names the net of Q3.1 (G), R25.2
- removed net LED_K: D9.2 (K), Q2.3 (C)
- net S4 renamed HV
- net HV: now also D8.1 (K); no longer D8.2 (K)
- net V3V3_SENSE: no longer names the net of U1.8 (PA7)
- new net: JP1.2 (B), R6.2
- no-connect marks 7 -> 9
Other:
- note added: "ARCHITECTURE ATtiny1616. PB2 PWM drives the boost. Counts stay on the MCU. Enable is firmware, not a pin. TTL is a test point. Power enters on STEMMA QT J4 and J5. No Pi header. No hardware OVP divider."
- note added: "BOOST AND MULTIPLIER"
- note added: "BOOST Q3 TN2404K-T1-GE3, 240 V, SOT-23. Pins 1 gate, 2 source, 3 drain. Gate is 3.3 V. L1 YNR6045-102M, 1 mH, 4.5 ohm. C1-C8 10 nF C0G 630 V. D1-D8 BAV21W. Footprint pad 1 is the cathode. Regulated window about 390-420 V. Switch node about 106 V there. 20% is a fault."
- note added: "PIN MAP PA0 UPDI. PA1 UART TX, USART0 alternate. PA2 collector. PA6 sense. PB2 HV_PWM. PB1 SDA. PB0 SCL. PC0 A0. PC1 A1. PA3 PA4 PA5 PA7 PB3 PB4 PB5 PC2 PC3 are no-connect. Default TX is PB2, so TX is remapped. TWI alternate is PA1/PA2 and is not used."
- note added: "POWER / I2C"
- note added: "SENSE AND TUBE R1-R4 33 MOhm 1% plus R5 412 kOhm 0.1%. PA6, VDD reference. About 1.04 V per count at the tube when VDD is 3.3 V. R11 R13 R15 R17 10 MOhm bleed HV to ground. R19 and R20 2.49 MOhm in series to the anode. D10 cathode clamps Q1 base. Clips are DNP. About 400 V. Discharge before handling."
- note added: "STEMMA QT J4 and J5, pin 1 GND, 2 3V3, 3 SDA, 4 SCL. JP2 and JP3 open: address 0x2F. A bridge pulls that address bit low. R26 and R27 are the only pull-ups."
- note added: "TUBE AND PULSE"
- note removed: "ARCHITECTURE ATtiny1616-only: MCU PWM drives HV boost, counts pulses, serves I2C, reads A0/A1 and HV/3V3 ADC. No TLC555 / MCP6562. Raw TTL pulse path stays hardware."
- note removed: "BOOST"
- note removed: "BOOST / HV Q3 HL2310A (1=G 2=S 3=D); R25 gate. L1 YNR6045-102M 1 mH, DCR 4.5 R. C1–C8: 10nF C0G 630V 1206. D1–D8: BAV21W. SW ~106 Vpk; S4 ~399 V."
- note removed: "DESIGN NOTES"
- note removed: "HV MULTIPLIER"
- note removed: "OUTPUT / LED"
- note removed: "OVP / PULSE / TUBE"
- note removed: "PI HEADER"
- note removed: "PIN MAP — U1 PA2 COLLECTOR PA4 SDA PA5 SCL PA6 SENSE (HV) PA7 V3V3_SENSE PB0 A0 PB1 A1 PB2 HV_PWM PB3 EN PA0 UPDI PA1 UART_TX (USART0 alt) Default USART0 TX is PB2 — remapped."
- note removed: "PROBE ACCESS"
- note removed: "SAFETY / FAB 400 V on tube clips / HV nodes. Discharge before handling. PCB: known DRC issues — prototype only. Clips C142864 DNP; fit after assembly. Run ERC; human-review HV creepage."
- note removed: "STEMMA / I2C"
- note removed: "STEMMA QT / ADDRESS J4/J5 JST-SH: 1=GND 2=3V3 3=SDA 4=SCL JP2/JP3 open = 0x2F; bridge = low bit. One pull-up set per bus segment."
- moved on the sheet: C1, C11, C2, C3, C4, C5, C6, C7, C8, C9, D1, D10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

Commit message: Point J4 and J5 at the SRSS land and correct C11.
The STEMMA connectors stay SM04B-SRSS-TB and now use the stock JST SH footprint. C11 stays 100 nF and is CL10B104KB8NNNC (LCSC C1591) on a 0603 land. The board file is unchanged. Notes record that BAV21W-7-F is a 200 V part and the deck's 250 V diode is generic.
Parts:
- C11: footprint glowcost:C1 -> Capacitor_SMD:C_0603_1608Metric; LCSC C342714 -> C1591; MPN C3216C0G2J103JT000N -> CL10B104KB8NNNC
- J4, J5: footprint glowcost:J1 -> Connector_JST:JST_SH_SM04B-SRSS-TB_1x04-1MP_P1.00mm_Horizontal
Changed lines of the file:
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@@
 (property
 "Footprint"
-"glowcost:J1"
+"Connector_JST:JST_SH_SM04B-SRSS-TB_1x04-1MP_P1.00mm_Horizontal"
 (at 38.1 35.56 0)
 (hide yes)
@@
 (property
 "Footprint"
-"glowcost:J1"
+"Connector_JST:JST_SH_SM04B-SRSS-TB_1x04-1MP_P1.00mm_Horizontal"
 (at 38.1 63.5 0)
 (hide yes)
@@
 (property
 "Footprint"
-"glowcost:C1"
+"Capacitor_SMD:C_0603_1608Metric"
 (at 137.16 52.07 0)
 (hide yes)
@@
 (property
 "Datasheet"
-""
+"https://www.lcsc.com/datasheet/C1591.pdf"
 (at 137.16 52.07 0)
 (hide yes)
@@
 (property
 "Description"
-""
+"100 nF 50 V X7R 0603"
 (at 137.16 52.07 0)
 (show_name no)
@@
 (property
 "MPN"
-"C3216C0G2J103JT000N"
+"CL10B104KB8NNNC"
 (at 137.16 52.07 0)
 (hide yes)
@@
 (property
 "LCSC"
-"C342714"
+"C1591"
 (at 137.16 52.07 0)
 (hide yes)

Commit message: Add the I2C slave and hold the boost off until enable.
CTC-5/STS-5 and SBM-20 share the ~400 V loop. Boot leaves PWM at zero until the host sets CTRL bit 0. Counts are a running total plus the previous second.
Parts:
- GM1: value CTC-5 / STS-5 -> STS-5 / SBM-20
Other:
- note added: "SENSE AND TUBE R1-R4 33 MOhm 1% plus R5 412 kOhm 0.1%. PA6, VDD reference. About 1.04 V per count at the tube when VDD is 3.3 V. R11 R13 R15 R17 10 MOhm bleed HV to ground. R19 and R20 2.49 MOhm in series to the anode. D10 cathode clamps Q1 base. Clips are DNP. CTC-5, STS-5, and SBM-20 share this bias. About 400 V. Discharge before handling."
- note removed: "SENSE AND TUBE R1-R4 33 MOhm 1% plus R5 412 kOhm 0.1%. PA6, VDD reference. About 1.04 V per count at the tube when VDD is 3.3 V. R11 R13 R15 R17 10 MOhm bleed HV to ground. R19 and R20 2.49 MOhm in series to the anode. D10 cathode clamps Q1 base. Clips are DNP. About 400 V. Discharge before handling."
Changed lines of the file:
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@@
 (property
 "Value"
-"CTC-5 / STS-5"
+"STS-5 / SBM-20"
 (at 63.5 172.72 0)
 (show_name no)
@@
 )
 (text
-"SENSE AND TUBE\n\nR1-R4 33 MOhm 1% plus R5 412 kOhm 0.1%.\nPA6, VDD reference. About 1.04 V per count\nat the tube when VDD is 3.3 V.\nR11 R13 R15 R17 10 MOhm bleed HV to ground.\nR19 and R20 2.49 MOhm in series to the anode.\nD10 cathode clamps Q1 base. Clips are DNP.\nAbout 400 V. Discharge before handling."
+"SENSE AND TUBE\n\nR1-R4 33 MOhm 1% plus R5 412 kOhm 0.1%.\nPA6, VDD reference. About 1.04 V per count\nat the tube when VDD is 3.3 V.\nR11 R13 R15 R17 10 MOhm bleed HV to ground.\nR19 and R20 2.49 MOhm in series to the anode.\nD10 cathode clamps Q1 base. Clips are DNP.\nCTC-5, STS-5, and SBM-20 share this bias.\nAbout 400 V. Discharge before handling."
 (at 165.1 254 0)
 (effects
