File: pcb/glowcost-geiger.kicad_sch (KiCad schematic)
At the start: 64 parts, among them J2 C142864 DNP, J3 C142864 DNP, J4 SM04B-SRSS-TB / C160404, J5 SM04B-SRSS-TB / C160404, Q1 MMBT3904LT1G, Q2 MMBT3904LT1G, Q3 TN2404K / C468011, U1 ATTINY1616-MNR / C507118

Commit message: Update the board for the SBM-20 and the firmware faults.
J2 and J3 are both C19184098. The ATtiny, boost switch, and STEMMA QT connectors sit on a bay added along the lower edge. Multiplier copper that still matched the sheet was kept; the new nets are not fully routed. Fault traces follow the PA6 trip and the 20% latch.
Parts:
- GM1: value STS-5 / SBM-20 -> SBM-20
- J2: value C142864 DNP -> C19184098; footprint glowcost:J2 -> MY-AA-03:MY-AA-03; symbol Glowcost:Conn_01x02 -> MY-AA-03:MY-AA-03; LCSC C142864 -> C19184098; MPN 10207101009 -> MY-AA-03; now fitted
- J3: value C142864 DNP -> C19184098; footprint glowcost:J3 -> MY-AA-03:MY-AA-03; symbol Glowcost:Conn_01x02 -> MY-AA-03:MY-AA-03; LCSC C142864 -> C19184098; MPN 10207101009 -> MY-AA-03; now fitted
Connections:
- net ANODE: no longer J2.2 (Pin_2)
- net CATHODE: no longer J3.2 (Pin_2)
Other:
- note added: "SENSE AND TUBE R1-R4 33 MOhm 1% plus R5 412 kOhm 0.1%. PA6, VDD reference. About 1.04 V per count at the tube when VDD is 3.3 V. R11 R13 R15 R17 10 MOhm bleed HV to ground. R19 and R20 2.49 MOhm in series to the anode. D10 cathode clamps Q1 base. SBM-20, about 108 mm. Both ends are C19184098 springs. A spacer holds the tube. About 400 V. Discharge before handling."
- note removed: "SENSE AND TUBE R1-R4 33 MOhm 1% plus R5 412 kOhm 0.1%. PA6, VDD reference. About 1.04 V per count at the tube when VDD is 3.3 V. R11 R13 R15 R17 10 MOhm bleed HV to ground. R19 and R20 2.49 MOhm in series to the anode. D10 cathode clamps Q1 base. Clips are DNP. CTC-5, STS-5, and SBM-20 share this bias. About 400 V. Discharge before handling."
Changed lines of the file:
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@@
 )
 (symbol
-(lib_id "Glowcost:Conn_01x02")
-(at 30.48 157.48 0)
+(lib_id "MY-AA-03:MY-AA-03")
+(at 22.86 158.75 0)
 (unit 1)
 (body_style 1)
@@
 (on_board yes)
 (in_pos_files yes)
-(dnp yes)
+(dnp no)
 (property
 "Reference"
 "J2"
-(at 30.48 151.13 0)
+(at 33.02 152.4 0)
 (show_name no)
 (do_not_autoplace no)
@@
 (property
 "Value"
-"C142864 DNP"
-(at 30.48 163.83 0)
+"C19184098"
+(at 33.02 155.0 0)
 (show_name no)
 (do_not_autoplace no)
@@
 (property
 "Footprint"
-"glowcost:J2"
-(at 30.48 157.48 0)
+"MY-AA-03:MY-AA-03"
+(at 22.86 158.75 0)
 (hide yes)
 (show_name no)
@@
 (property
 "Datasheet"
-""
-(at 30.48 157.48 0)
+"${KIPRJMOD}/components/MY-AA-03/MY-AA-03.pdf"
+(at 22.86 158.75 0)
 (hide yes)
 (show_name no)
@@
 (property
 "Description"
-""
-(at 30.48 157.48 0)
+"SMD negative spring, both tube ends"
+(at 22.86 158.75 0)
 (show_name no)
 (do_not_autoplace no)
@@
 (property
 "MPN"
-"10207101009"
-(at 30.48 157.48 0)
+"MY-AA-03"
+(at 22.86 158.75 0)
 (hide yes)
 (show_name no)
@@
 (property
 "LCSC"
-"C142864"
-(at 30.48 157.48 0)
+"C19184098"
+(at 22.86 158.75 0)
 (hide yes)
 (show_name no)
@@
 "1"
 )
-(pin
-"2"
-)
 (instances
 (project
@@
 )
 (symbol
-(lib_id "Glowcost:Conn_01x02")
-(at 30.48 175.26 0)
+(lib_id "MY-AA-03:MY-AA-03")
+(at 22.86 176.53 0)
 (unit 1)
 (body_style 1)
@@
 (on_board yes)
 (in_pos_files yes)
-(dnp yes)
+(dnp no)
 (property
 "Reference"
 "J3"
-(at 30.48 168.91 0)
+(at 33.02 170.18 0)
 (show_name no)
 (do_not_autoplace no)
@@
 (property
 "Value"
-"C142864 DNP"
-(at 30.48 181.61 0)
+"C19184098"
+(at 33.02 172.72 0)
 (show_name no)
 (do_not_autoplace no)
@@
 (property
 "Footprint"
-"glowcost:J3"
-(at 30.48 175.26 0)
+"MY-AA-03:MY-AA-03"
+(at 22.86 176.53 0)
 (hide yes)
 (show_name no)
@@
 (property
 "Datasheet"
-""
-(at 30.48 175.26 0)
+"${KIPRJMOD}/components/MY-AA-03/MY-AA-03.pdf"
+(at 22.86 176.53 0)
 (hide yes)
 (show_name no)
@@
 (property
 "Description"
-""
-(at 30.48 175.26 0)
+"SMD negative spring, both tube ends"
+(at 22.86 176.53 0)
 (show_name no)
 (do_not_autoplace no)
@@
 (property
 "MPN"
-"10207101009"
-(at 30.48 175.26 0)
+"MY-AA-03"
+(at 22.86 176.53 0)
 (hide yes)
 (show_name no)
@@
 (property
 "LCSC"
-"C142864"
-(at 30.48 175.26 0)
+"C19184098"
+(at 22.86 176.53 0)
 (hide yes)
 (show_name no)
@@
 "1"
 )
-(pin
-"2"
-)
 (instances
 (project
@@
 (wire
 (pts
-(xy 25.4 157.48)
-(xy 20.32 157.48)
-)
-(stroke
-(width 0.1524)
-(type default)
-(color 160 40 40 1)
-)
-)
-(wire
-(pts
-(xy 25.4 160.02)
-(xy 20.32 160.02)
-)
-(stroke
-(width 0.1524)
-(type default)
-(color 160 40 40 1)
-)
-)
-(wire
-(pts
-(xy 20.32 157.48)
-(xy 20.32 160.02)
-)
-(stroke
-(width 0.1524)
-(type default)
-(color 160 40 40 1)
-)
-)
-(wire
-(pts
 (xy 20.32 158.75)
 (xy 15.24 158.75)
@@
 (color 0 0 0 0)
 )
-(junction
-(at 20.32 157.48)
-(diameter 0)
-(color 0 0 0 0)
-)
-(junction
-(at 20.32 160.02)
-(diameter 0)
-(color 0 0 0 0)
-)
-(wire
-(pts
-(xy 25.4 175.26)
-(xy 20.32 175.26)
-)
-(stroke
-(width 0.1524)
-(type default)
-(color 60 80 80 1)
-)
-)
-(wire
-(pts
-(xy 25.4 177.8)
-(xy 20.32 177.8)
-)
-(stroke
-(width 0.1524)
-(type default)
-(color 60 80 80 1)
-)
-)
-(wire
-(pts
-(xy 20.32 175.26)
-(xy 20.32 177.8)
-)
-(stroke
-(width 0.1524)
-(type default)
-(color 60 80 80 1)
-)
-)
 (wire
 (pts
@@
 (color 0 0 0 0)
 )
-(junction
-(at 20.32 175.26)
-(diameter 0)
-(color 0 0 0 0)
-)
-(junction
-(at 20.32 177.8)
-(diameter 0)
-(color 0 0 0 0)
-)
 (symbol
 (lib_id "Glowcost:SparkGap")
@@
 (property
 "Value"
-"STS-5 / SBM-20"
+"SBM-20"
 (at 63.5 172.72 0)
 (show_name no)
@@
 )
 (text
-"SENSE AND TUBE\n\nR1-R4 33 MOhm 1% plus R5 412 kOhm 0.1%.\nPA6, VDD reference. About 1.04 V per count\nat the tube when VDD is 3.3 V.\nR11 R13 R15 R17 10 MOhm bleed HV to ground.\nR19 and R20 2.49 MOhm in series to the anode.\nD10 cathode clamps Q1 base. Clips are DNP.\nCTC-5, STS-5, and SBM-20 share this bias.\nAbout 400 V. Discharge before handling."
+"SENSE AND TUBE\n\nR1-R4 33 MOhm 1% plus R5 412 kOhm 0.1%.\nPA6, VDD reference. About 1.04 V per count\nat the tube when VDD is 3.3 V.\nR11 R13 R15 R17 10 MOhm bleed HV to ground.\nR19 and R20 2.49 MOhm in series to the anode.\nD10 cathode clamps Q1 base.\nSBM-20, about 108 mm. Both ends are\nC19184098 springs. A spacer holds the tube.\nAbout 400 V. Discharge before handling."
 (at 165.1 254 0)
 (effects
